Commit message: Fixed force sensor coordinates and added fse103_node to the launch file

File: urdf/slidertable.urdf (robot description, URDF)
Before this commit: robot slidertable, 3 links, 2 joints
Joints:
- joint slider_to_fs1: origin xyz=0 0.25 0.025 -> xyz=0 0.25 0.025 rpy=3.14 0 -1.57

Commit message: Added phidgets encoder to launch file with proper scale and fixed coordinate systems

File: urdf/slidertable.urdf (robot description, URDF)
Before this commit: robot slidertable, 3 links, 2 joints
Joints:
- joint slider_to_fs1: origin xyz=0 0.25 0.025 rpy=3.14 0 -1.57 -> xyz=0 -0.25 0.025 rpy=3.14 0 1.57
- joint tabletop_to_slider: origin xyz=0 0 0.025 -> xyz=0 0 0.025 rpy=0 0 3.14

Commit message: Updated urdf for new table construction. Needs load cell nodes.

File: urdf/slidertable.urdf (robot description, URDF)
Before this commit: robot slidertable, 3 links, 2 joints
Links:
- removed link force_sensor_1
- added link ball_knob_1; visual sphere radius=0.024
- added link ball_knob_2; visual sphere radius=0.024
- added link baseboard; visual box size=0.1778 0.4826 0.01905
- added link encoders
- link slider: geometry visual box size=0.1524 0.762 0.01905
Joints:
- removed joint slider_to_fs1
- removed joint tabletop_to_slider
- added joint baseboard_to_encoders: type prismatic, parent baseboard, child encoders, origin xyz=0 0 0 rpy=0 0 0, axis 0 1 0, limit lower=-0.3 upper=0.3 effort=1000.0 velocity=0.5
- added joint encoders_to_slider: type prismatic, parent encoders, child slider, origin xyz=0 0 0.028575 rpy=0 0 0, axis 0 1 0, limit lower=-0.3 upper=0.3 effort=1000.0 velocity=0.5
- added joint slider_to_knob1: type fixed, parent slider, child ball_knob_1, origin xyz=0 -0.43 0.0381 rpy=3.14 0 1.57
- added joint slider_to_knob2: type fixed, parent slider, child ball_knob_2, origin xyz=0 0.43 0.0381 rpy=3.14 0 -1.57
- added joint tabletop_to_baseboard: type fixed, parent tabletop, child baseboard, origin xyz=0 0 0.022 rpy=0 0 3.14

Commit message: Updated urdf and launch file for new encoder and motor system

File: urdf/slidertable.urdf (robot description, URDF)
Before this commit: robot slidertable, 6 links, 5 joints
Links:
- removed link encoders
Joints:
- removed joint baseboard_to_encoders
- removed joint encoders_to_slider
- added joint baseboard_to_slider: type prismatic, parent baseboard, child slider, origin xyz=0 0 0.028575 rpy=0 0 0, axis 0 1 0, limit lower=-0.3 upper=0.3 effort=1000.0 velocity=0.5

Commit message: Added second simulated slider urdf definitions and launch

File: urdf/slidertable.urdf (robot description, URDF)
Before this commit: robot slidertable, 5 links, 4 joints
Links:
- added link simslider; visual box size=0.1524 0.762 0.01905
Joints:
- added joint baseboard_to_simslider: type prismatic, parent baseboard, child simslider, origin xyz=0 0 0.028575 rpy=0 0 0, axis 0 1 0, limit lower=-0.3 upper=0.3 effort=1000.0 velocity=0.5
